Commit message: Updates to get working on russell

File: xacro/gummi_ee.srdf.xacro (robot description, xacro)
@@ -8,5 +8,5 @@
 <xacro:macro name="group_right_gripper_ee">
   <group name="right_gripper">
-      <link name="wrist" />
+      <link name="wrist_pitch" />
       <link name="gripper_Link" />
   </group>
@@ -26,8 +26,8 @@
   <disable_collisions link1="gripper_Link" link2="lowerarm" reason="Never" />
   <disable_collisions link1="gripper_Link" link2="lowerarm_preroll" reason="Never" />
-  <disable_collisions link1="gripper_Link" link2="wrist" reason="Adjacent" />
+  <disable_collisions link1="gripper_Link" link2="wrist_pitch" reason="Adjacent" />
   <disable_collisions link1="lowerarm" link2="lowerarm_preroll" reason="Adjacent" />
   <disable_collisions link1="lowerarm" link2="wrist" reason="Adjacent" />
-  <disable_collisions link1="lowerarm_preroll" link2="wrist" reason="Never" />
+  <disable_collisions link1="lowerarm_preroll" link2="wrist_pitch" reason="Never" />
 </xacro:macro>
 </robot>
