Commit message: Updating to make stls match what is real

File: xacro/gummi_description_ee.urdf.xacro (robot description, xacro)
@@ -47,6 +47,6 @@
     type="revolute">
     <origin
-      xyz="0 0 -0.1898"
-      rpy="0 0 0" />
+      xyz="0.008 -0.019 0.1896"
+      rpy="-1.57 0 3.14" />
     <parent
       link="upperarm" />
@@ -108,6 +108,6 @@
     type="revolute">
     <origin
-      xyz="0.0795 0.00025 -0.025"
-      rpy="0 0 0" />
+      xyz=" 0.08087 -0.026 -0.02075"
+      rpy="0 -1.57 -3.14" />
     <parent
       link="lowerarm_preroll" />
@@ -169,6 +169,6 @@
     type="revolute">
     <origin
-      xyz="0.084137 0 0.009003"
-      rpy="0 0 0" />
+      xyz="0.0191 -0.005 0.148"
+      rpy="0 -1.57 3.14" />
     <parent
       link="lowerarm" />
@@ -185,5 +185,5 @@
   </joint>
   <!-- gripper_Link -->
-  <link
+  <!-- <link
     name="gripper_Link">
     <inertial>
@@ -205,4 +205,8 @@
         xyz="0 0 0"
         rpy="0 0 0" />
+        <geometry>
+          <mesh
+            filename="package://gummi_base_template/meshes/gripper_Link.stl" />
+        </geometry>
       <material
         name="">
@@ -220,7 +224,7 @@
       </geometry>
     </collision>
-  </link>
+  </link> -->
   <!-- gripper -->
-  <joint
+  <!-- <joint
     name="gripper"
     type="revolute">
@@ -233,5 +237,5 @@
       link="gripper_Link" />
     <axis
-      xyz="0 1 0" />
+      xyz="0 1 0" /> -->
     <!-- <limit
       lower="-1.5708"
@@ -239,5 +243,5 @@
       effort="0"
       velocity="0" /> -->
-    <limit effort="0" lower="-0.30" upper="0.17" velocity="1.0"/>
-  </joint>
+    <!-- <limit effort="0" lower="-0.30" upper="0.17" velocity="1.0"/> -->
+  <!-- </joint> -->
 </robot>

File: xacro/gummi_ee.srdf.xacro (robot description, xacro)
@@ -9,5 +9,5 @@
   <group name="right_gripper">
       <link name="wrist_pitch" />
-      <link name="gripper_Link" />
+      <!-- <link name="gripper_Link" /> -->
   </group>
 </xacro:macro>
@@ -17,14 +17,14 @@
   <joint name="wrist_pitch" value="0" />
 </xacro:macro>
-<xacro:macro name="end_effector_ee">
+<!-- <xacro:macro name="end_effector_ee"> -->
   <!--END EFFECTOR: Purpose: Represent information about an end effector.-->
-  <end_effector name="right_eef" parent_link="wrist" group="right_gripper" />
-</xacro:macro>
+  <!-- <end_effector name="right_eef" parent_link="wrist" group="right_gripper" />
+</xacro:macro> -->
 <xacro:macro name="disable_collisions_ee">
   <!-- <disable_collisions link1="right_hand" link2="wrist" reason="Never" />
   <disable_collisions link1="right_hand" link2="gripper_Link" reason="Never" /> -->
-  <disable_collisions link1="gripper_Link" link2="lowerarm" reason="Never" />
+  <!-- <disable_collisions link1="gripper_Link" link2="lowerarm" reason="Never" />
   <disable_collisions link1="gripper_Link" link2="lowerarm_preroll" reason="Never" />
-  <disable_collisions link1="gripper_Link" link2="wrist_pitch" reason="Adjacent" />
+  <disable_collisions link1="gripper_Link" link2="wrist_pitch" reason="Adjacent" /> -->
   <disable_collisions link1="lowerarm" link2="lowerarm_preroll" reason="Adjacent" />
   <disable_collisions link1="lowerarm" link2="wrist" reason="Adjacent" />

Commit message: URDF Changes

File: xacro/gummi_description_ee.urdf.xacro (robot description, xacro)
@@ -185,5 +185,5 @@
   </joint>
   <!-- gripper_Link -->
-  <!-- <link
+  <link
     name="gripper_Link">
     <inertial>
@@ -224,12 +224,12 @@
       </geometry>
     </collision>
-  </link> -->
+  </link>
   <!-- gripper -->
-  <!-- <joint
+  <joint
     name="gripper"
     type="revolute">
     <origin
-      xyz="0.066697 -0.0261 0.0093282"
-      rpy="1.5708 1.0472 3.1416" />
+      xyz="0.028 0 -0.02075"
+      rpy="0 -1.57 3.14" />
     <parent
       link="wrist" />
@@ -237,5 +237,5 @@
       link="gripper_Link" />
     <axis
-      xyz="0 1 0" /> -->
+      xyz="0 0 1" />
     <!-- <limit
       lower="-1.5708"
@@ -243,5 +243,5 @@
       effort="0"
       velocity="0" /> -->
-    <!-- <limit effort="0" lower="-0.30" upper="0.17" velocity="1.0"/> -->
-  <!-- </joint> -->
+    <limit effort="0" lower="-0.30" upper="0.17" velocity="1.0"/>
+  </joint>
 </robot>

File: xacro/gummi_ee.srdf.xacro (robot description, xacro)
@@ -8,6 +8,6 @@
 <xacro:macro name="group_right_gripper_ee">
   <group name="right_gripper">
-      <link name="wrist_pitch" />
-      <!-- <link name="gripper_Link" /> -->
+      <link name="wrist" />
+      <link name="gripper_Link" />
   </group>
 </xacro:macro>
@@ -17,17 +17,17 @@
   <joint name="wrist_pitch" value="0" />
 </xacro:macro>
-<!-- <xacro:macro name="end_effector_ee"> -->
+<xacro:macro name="end_effector_ee">
   <!--END EFFECTOR: Purpose: Represent information about an end effector.-->
-  <!-- <end_effector name="right_eef" parent_link="wrist" group="right_gripper" />
-</xacro:macro> -->
+  <end_effector name="right_eef" parent_link="wrist" group="right_gripper" />
+</xacro:macro>
 <xacro:macro name="disable_collisions_ee">
-  <!-- <disable_collisions link1="right_hand" link2="wrist" reason="Never" />
-  <disable_collisions link1="right_hand" link2="gripper_Link" reason="Never" /> -->
-  <!-- <disable_collisions link1="gripper_Link" link2="lowerarm" reason="Never" />
+  <disable_collisions link1="right_hand" link2="wrist" reason="Never" />
+  <disable_collisions link1="right_hand" link2="gripper_Link" reason="Never" />
+  <disable_collisions link1="gripper_Link" link2="lowerarm" reason="Never" />
   <disable_collisions link1="gripper_Link" link2="lowerarm_preroll" reason="Never" />
-  <disable_collisions link1="gripper_Link" link2="wrist_pitch" reason="Adjacent" /> -->
+  <disable_collisions link1="gripper_Link" link2="wrist" reason="Adjacent" />
   <disable_collisions link1="lowerarm" link2="lowerarm_preroll" reason="Adjacent" />
   <disable_collisions link1="lowerarm" link2="wrist" reason="Adjacent" />
-  <disable_collisions link1="lowerarm_preroll" link2="wrist_pitch" reason="Never" />
+  <disable_collisions link1="lowerarm_preroll" link2="wrist" reason="Never" />
 </xacro:macro>
 </robot>

Commit message: Made necessary changes for Luffy

File: xacro/gummi_description_ee.urdf.xacro (robot description, xacro)
@@ -23,19 +23,19 @@
       <geometry>
         <mesh
-          filename="package://gummi_ee_$(env ROS_GUMMI_EE)/meshes/lowerarm_preroll_d.STL" />
-      </geometry>
-      <material
-        name="">
-        <color
-          rgba="0.792156862745098 0.819607843137255 0.933333333333333 1" />
-      </material>
-    </visual>
-    <collision>
-      <origin
-        xyz="0 0 0"
-        rpy="0 0 0" />
-      <geometry>
-        <mesh
-          filename="package://gummi_ee_$(env ROS_GUMMI_EE)/meshes/lowerarm_preroll_d.STL" />
+          filename="package://gummi_ee_$(env ROS_GUMMI_EE)/meshes/j5_Link.stl" />
+      </geometry>
+      <material
+        name="">
+        <color
+          rgba="0.792156862745098 0.819607843137255 0.933333333333333 1" />
+      </material>
+    </visual>
+    <collision>
+      <origin
+        xyz="0 0 0"
+        rpy="0 0 0" />
+      <geometry>
+        <mesh
+          filename="package://gummi_ee_$(env ROS_GUMMI_EE)/meshes/j5_Link.stl" />
       </geometry>
     </collision>
@@ -76,19 +76,19 @@
       <geometry>
         <mesh
-          filename="package://gummi_ee_$(env ROS_GUMMI_EE)/meshes/lowerarm.STL" />
-      </geometry>
-      <material
-        name="">
-        <color
-          rgba="0.792156862745098 0.819607843137255 0.933333333333333 1" />
-      </material>
-    </visual>
-    <collision>
-      <origin
-        xyz="0 0 0"
-        rpy="0 0 0" />
-      <geometry>
-        <mesh
-          filename="package://gummi_ee_$(env ROS_GUMMI_EE)/meshes/lowerarm.STL" />
+          filename="package://gummi_ee_$(env ROS_GUMMI_EE)/meshes/j6_link.stl" />
+      </geometry>
+      <material
+        name="">
+        <color
+          rgba="0.792156862745098 0.819607843137255 0.933333333333333 1" />
+      </material>
+    </visual>
+    <collision>
+      <origin
+        xyz="0 0 0"
+        rpy="0 0 0" />
+      <geometry>
+        <mesh
+          filename="package://gummi_ee_$(env ROS_GUMMI_EE)/meshes/j6_link.stl" />
       </geometry>
     </collision>
@@ -132,19 +132,19 @@
       <geometry>
         <mesh
-          filename="package://gummi_ee_$(env ROS_GUMMI_EE)/meshes/wrist.STL" />
-      </geometry>
-      <material
-        name="">
-        <color
-          rgba="0.792156862745098 0.819607843137255 0.933333333333333 1" />
-      </material>
-    </visual>
-    <collision>
-      <origin
-        xyz="0 0 0"
-        rpy="0 0 0" />
-      <geometry>
-        <mesh
-          filename="package://gummi_ee_$(env ROS_GUMMI_EE)/meshes/wrist.STL" />
+          filename="package://gummi_ee_$(env ROS_GUMMI_EE)/meshes/j7_Link.stl" />
+      </geometry>
+      <material
+        name="">
+        <color
+          rgba="0.792156862745098 0.819607843137255 0.933333333333333 1" />
+      </material>
+    </visual>
+    <collision>
+      <origin
+        xyz="0 0 0"
+        rpy="0 0 0" />
+      <geometry>
+        <mesh
+          filename="package://gummi_ee_$(env ROS_GUMMI_EE)/meshes/j7_Link.stl" />
       </geometry>
     </collision>

Commit message: Created custom EE for Luffy
Includes Bi-Directional Wrist with AX Motors

File: xacro/gummi_description_ee.urdf.xacro (robot description, xacro)
@@ -23,19 +23,19 @@
       <geometry>
         <mesh
-          filename="package://gummi_ee_$(env ROS_GUMMI_EE)/meshes/j5_Link.stl" />
-      </geometry>
-      <material
-        name="">
-        <color
-          rgba="0.792156862745098 0.819607843137255 0.933333333333333 1" />
-      </material>
-    </visual>
-    <collision>
-      <origin
-        xyz="0 0 0"
-        rpy="0 0 0" />
-      <geometry>
-        <mesh
-          filename="package://gummi_ee_$(env ROS_GUMMI_EE)/meshes/j5_Link.stl" />
+          filename="package://gummi_ee_$(env ROS_GUMMI_EE)/meshes/lowerarm_preroll_d.stl" />
+      </geometry>
+      <material
+        name="">
+        <color
+          rgba="0.792156862745098 0.819607843137255 0.933333333333333 1" />
+      </material>
+    </visual>
+    <collision>
+      <origin
+        xyz="0 0 0"
+        rpy="0 0 0" />
+      <geometry>
+        <mesh
+          filename="package://gummi_ee_$(env ROS_GUMMI_EE)/meshes/lowerarm_preroll_d_CH.stl" />
       </geometry>
     </collision>
@@ -45,6 +45,6 @@
     type="fixed">
     <origin
-      xyz="0.056236 -0.019 -0.006"
-      rpy="0 0 0" />
+      xyz="0.00037 0.102 -0.02055"
+      rpy="1.57 -1.57 0" />
     <parent
       link="lowerarm_preroll_u" />
@@ -90,5 +90,5 @@
       <geometry>
         <mesh
-          filename="package://gummi_ee_$(env ROS_GUMMI_EE)/meshes/j6_link.stl" />
+          filename="package://gummi_ee_$(env ROS_GUMMI_EE)/meshes/j6_link_CH.stl" />
       </geometry>
     </collision>
@@ -98,6 +98,6 @@
     type="continuous">
     <origin
-      xyz="0.043506 -0.00023376 -0.019876"
-      rpy="0 0 0" />
+      xyz="0 0 0.04"
+      rpy="0 0 3.16" />
     <parent
       link="lowerarm_preroll_d" />
@@ -105,5 +105,5 @@
       link="lowerarm" />
     <axis
-      xyz="-1 0 0" />
+      xyz="0 0 1" />
     <limit
       effort="0"
@@ -146,5 +146,5 @@
       <geometry>
         <mesh
-          filename="package://gummi_ee_$(env ROS_GUMMI_EE)/meshes/j7_Link.stl" />
+          filename="package://gummi_ee_$(env ROS_GUMMI_EE)/meshes/j7_Link_CH.stl" />
       </geometry>
     </collision>
@@ -154,6 +154,6 @@
     type="revolute">
     <origin
-      xyz="0.1511 -0.01935 0.0048471"
-      rpy="0 0 0" />
+      xyz="0.0192 0 -0.16357"
+      rpy="0 1.57 0" />
     <parent
       link="lowerarm" />
@@ -161,5 +161,5 @@
       link="wrist" />
     <axis
-      xyz="0 1 0" />
+      xyz="0 0 -1" />
     <limit
       lower="-1"
@@ -173,5 +173,5 @@
   offset and a multiplication rate. check ros docs for details
   -->
-  <joint name="gripper" type="revolute">
+  <!-- <joint name="gripper" type="revolute">
     <origin rpy="0 0 0" xyz="0 0 0"/>
     <parent link="wrist"/>
@@ -475,4 +475,4 @@
       velocity="0" />
     <mimic joint="gripper"/>
-  </joint>
+  </joint> -->
 </robot>

File: xacro/gummi_ee.srdf.xacro (robot description, xacro)
@@ -5,41 +5,9 @@
     <joint name="wrist_pitch" />
 </xacro:macro>
-<xacro:macro name="group_right_gripper_ee">
-  <group name="right_gripper">
-    <link name="wrist"/>
-    <joint name="gripper"/>
-  </group>
-</xacro:macro>
 <xacro:macro name="group_state_right_arm_ee">
   <joint name="forearm_roll" value="0" />
   <joint name="wrist_pitch" value="0" />
 </xacro:macro>
-<xacro:macro name="end_effector_ee">
-  <!--END EFFECTOR: Purpose: Represent information about an end effector.-->
-<end_effector group="right_gripper" name="right_eef" parent_link="wrist" parent_group="right_arm"/>
-</xacro:macro>
 <xacro:macro name="disable_collisions_ee">
-  <!-- <disable_collisions link1="right_hand" link2="wrist" reason="Never" />
-  <disable_collisions link1="right_hand" link2="gripper_link" reason="Never" /> -->
-  <disable_collisions link1="i1" link2="lowerarm" reason="Never" />
-  <disable_collisions link1="i2" link2="lowerarm" reason="Never" />
-  <disable_collisions link1="i3" link2="lowerarm" reason="Never" />
-  <disable_collisions link1="i4" link2="lowerarm" reason="Never" />
-  <disable_collisions link1="i5" link2="lowerarm" reason="Never" />
-  <disable_collisions link1="i1" link2="wrist" reason="Never" />
-  <disable_collisions link1="i2" link2="wrist" reason="Never" />
-  <disable_collisions link1="i3" link2="wrist" reason="Never" />
-  <disable_collisions link1="i4" link2="wrist" reason="Never" />
-  <disable_collisions link1="i5" link2="wrist" reason="Never" />
-  <disable_collisions link1="i1" link2="i2" reason="Never" />
-  <disable_collisions link1="i1" link2="i3" reason="Never" />
-  <disable_collisions link1="i1" link2="i4" reason="Never" />
-  <disable_collisions link1="i1" link2="i5" reason="Never" />
-  <disable_collisions link1="i2" link2="i3" reason="Never" />
-  <disable_collisions link1="i2" link2="i4" reason="Never" />
-  <disable_collisions link1="i2" link2="i5" reason="Never" />
-  <disable_collisions link1="i3" link2="i4" reason="Never" />
-  <disable_collisions link1="i3" link2="i5" reason="Never" />
-  <disable_collisions link1="i4" link2="i5" reason="Never" />
   <disable_collisions link1="lowerarm" link2="lowerarm_preroll_d" reason="Adjacent" />
   <disable_collisions link1="lowerarm" link2="wrist" reason="Adjacent" />

Commit message: Added Pointer end effector and fixed transforms

File: xacro/gummi_description_ee.urdf.xacro (robot description, xacro)
@@ -45,6 +45,6 @@
     type="fixed">
     <origin
-      xyz="0.00037 0.102 -0.02055"
-      rpy="1.57 -1.57 0" />
+      xyz="0.00037 0.10187 -0.021"
+      rpy="1.57079632679 -1.57079632679 0" />
     <parent
       link="lowerarm_preroll_u" />
@@ -98,6 +98,6 @@
     type="continuous">
     <origin
-      xyz="0 0 0.04"
-      rpy="0 0 3.16" />
+      xyz="0 0 0.03987"
+      rpy="0 0 3.14159265359" />
     <parent
       link="lowerarm_preroll_d" />
@@ -105,5 +105,5 @@
       link="lowerarm" />
     <axis
-      xyz="0 0 1" />
+      xyz="0 0 -1" />
     <limit
       effort="0"
@@ -154,6 +154,6 @@
     type="revolute">
     <origin
-      xyz="0.0192 0 -0.16357"
-      rpy="0 1.57 0" />
+      xyz="0.019 0 -0.16357"
+      rpy="0 1.57079632679 0" />
     <parent
       link="lowerarm" />
@@ -167,4 +167,57 @@
       effort="0"
       velocity="0" />
+  </joint>
+    <link
+    name="pointer">
+    <inertial>
+      <origin
+        xyz="0.0484512742480244 0.0139768664666073 0.000956995637939325"
+        rpy="0 0 0" />
+      <mass
+        value="0.0644774651698934" />
+      <inertia
+        ixx="8.67406414845019E-06"
+        ixy="-1.3193756197629E-05"
+        ixz="-3.41916035169704E-06"
+        iyy="4.217442276821E-05"
+        iyz="-4.04257224014858E-07"
+        izz="4.91399139463636E-05" />
+    </inertial>
+    <visual>
+      <origin
+        xyz="0 0 0"
+        rpy="0 0 0" />
+      <geometry>
+        <mesh
+          filename="package://gummi_ee_$(env ROS_GUMMI_EE)/meshes/pointer_gripper.stl" />
+      </geometry>
+      <material
+        name="">
+        <color
+          rgba="0.792156862745098 0.819607843137255 0.933333333333333 1" />
+      </material>
+    </visual>
+    <collision>
+      <origin
+        xyz="0 0 0"
+        rpy="0 0 0" />
+      <geometry>
+        <mesh
+          filename="package://gummi_ee_$(env ROS_GUMMI_EE)/meshes/pointer_gripper_CH.stl" />
+      </geometry>
+    </collision>
+  </link>
+  <joint
+    name="end_effector"
+    type="fixed">
+    <origin
+      xyz="0.0966 0 -0.0202"
+      rpy="0 1.57079632679 0" />
+    <parent
+      link="wrist" />
+    <child
+      link="pointer" />
+    <axis
+      xyz="0 0 0" />
   </joint>
   <!--

File: xacro/gummi_ee.srdf.xacro (robot description, xacro)
@@ -4,4 +4,7 @@
     <joint name="forearm_roll" />
     <joint name="wrist_pitch" />
+</xacro:macro>
+<xacro:macro name="group_pointer">
+    <joint name="end_effector" />
 </xacro:macro>
 <xacro:macro name="group_state_right_arm_ee">

Commit message: Updated Gripper

File: xacro/gummi_description_ee.urdf.xacro (robot description, xacro)
@@ -190,19 +190,19 @@
       <geometry>
         <mesh
-          filename="package://gummi_ee_$(env ROS_GUMMI_EE)/meshes/pointer_gripper.stl" />
-      </geometry>
-      <material
-        name="">
-        <color
-          rgba="0.792156862745098 0.819607843137255 0.933333333333333 1" />
-      </material>
-    </visual>
-    <collision>
-      <origin
-        xyz="0 0 0"
-        rpy="0 0 0" />
-      <geometry>
-        <mesh
-          filename="package://gummi_ee_$(env ROS_GUMMI_EE)/meshes/pointer_gripper_CH.stl" />
+          filename="package://gummi_ee_$(env ROS_GUMMI_EE)/meshes/pointer_gripper_EIH.stl" />
+      </geometry>
+      <material
+        name="">
+        <color
+          rgba="0.792156862745098 0.819607843137255 0.933333333333333 1" />
+      </material>
+    </visual>
+    <collision>
+      <origin
+        xyz="0 0 0"
+        rpy="0 0 0" />
+      <geometry>
+        <mesh
+          filename="package://gummi_ee_$(env ROS_GUMMI_EE)/meshes/pointer_gripper_EIH_CH.stl" />
       </geometry>
     </collision>
@@ -213,5 +213,5 @@
     <origin
       xyz="0.0966 0 -0.0202"
-      rpy="0 1.57079632679 0" />
+      rpy="0 -1.57079632679 3.14159265359" />
     <parent
       link="wrist" />
